File: boards/EmbeddedKeyboard/EmbeddedKeyboard.kicad_sch (KiCad schematic)
At the start: 41 parts, among them J1 S2B-PH-SM4-TB, J2 Conn_01x20_Pin, J8 USB_C_Receptacle_USB2.0_14P, Q1 DMN3135LVT-7, SW1 SLIDE SWITCH, U1 LM3671MFX-3.3_NOPB, U2 MCP73831T-2ACI_OT, U3 ESP32-WROOM-32E, U5 CH340C

Commit message: Enough spec to communicate intent
Parts:
- removed J2: Conn_01x20_Pin, Connector_PinHeader_2.54mm:PinHeader_1x20_P2.54mm_Vertical, symbol Connector:Conn_01x20_Pin
- removed SW1: SLIDE SWITCH, JS202011SCQN:JS202011SCQN, symbol JS202011SCQN:JS202011SCQN
- added C1, C10, C11, C12, C13, C14, C15, C2, C24, C25, C26, C27, C28, C29, C3, C30, C31, C32, C33, C34, C35, C36, C37, C38, C39, C4, C40, C41, C42, C43, C44, C45, C46, C47, C48, C49, C5, C52, C53, C54, C55, C56, C57, C58, C59, C6, C60, C61, C62, C7, C8, C9: 100nF, CAP_CL03_SAM, symbol CL03A104KP3NNNC:CL03A104KP3NNNC
- added H1, H2, H3, H4, H5, H6, H7: MountingHole, symbol Mechanical:MountingHole
- added J2: EXTERNAL SWITCH, S2B-PH-SM4-TB:S2B-PH-SM4-TB, symbol S2B-PH-SM4-TB:S2B-PH-SM4-TB
- added R20, R21, R24, R25, R28, R29, R3, R30, R4, R5: 10K, Resistor_SMD:R_0402_1005Metric, symbol Device:R
- added R22, R23, R26, R27, R31, R32, R33, R34, R35, R36, R37, R38, R39, R40, R41, R42, R43, R44, R45, R46, R47, R48, R49, R50, R51, R52: 75K, RT0805FRE0775KL:RESC2012X60N, symbol RT0805FRE0775KL:RT0805FRE0775KL
- added TP1, TP10, TP100, TP101, TP102, TP103, TP104, TP105, TP106, TP107, TP108, TP109, TP11, TP110, TP111, TP112, TP113, TP114, TP115, TP116, TP117, TP118, TP119, TP12, TP120, TP121, TP122, TP123, TP124, TP125, TP126, TP127, TP128, TP129, TP13, TP130, TP131, TP132, TP133, TP134, TP135, TP136, TP137, TP138, TP139, TP14, TP140, TP141, TP142, TP143, TP144, TP145, TP146, TP147, TP148, TP149, TP15, TP150, TP151, TP152, TP153, TP154, TP155, TP156, TP157, TP158, TP159, TP16, TP160, TP161, TP162, TP163, TP164, TP165, TP166, TP167, TP168, TP169, TP17, TP170, TP171, TP172, TP173, TP174, TP175, TP176, TP177, TP178, TP179, TP18, TP180, TP181, TP182, TP183, TP184, TP185, TP186, TP187, TP188, TP189, TP19, TP190, TP191, TP192, TP193, TP194, TP195, TP196, TP197, TP198, TP199, TP2, TP20, TP200, TP201, TP202, TP203, TP204, TP205, TP206, TP207, TP208, TP209, TP21, TP210, TP211, TP212, TP213, TP214, TP215, TP216, TP217, TP218, TP219, TP22, TP220, TP221, TP222, TP223, TP224, TP225, TP226, TP227, TP228, TP229, TP23, TP230, TP231, TP232, TP233, TP234, TP235, TP236, TP237, TP238, TP239, TP24, TP240, TP241, TP242, TP243, TP244, TP245, TP246, TP247, TP248, TP249, TP25, TP250, TP251, TP252, TP253, TP254, TP255, TP256, TP257, TP258, TP259, TP26, TP260, TP261, TP262, TP263, TP264, TP265, TP266, TP267, TP268, TP269, TP27, TP270, TP271, TP272, TP273, TP274, TP275, TP276, TP277, TP278, TP279, TP28, TP280, TP281, TP282, TP283, TP284, TP285, TP286, TP287, TP288, TP289, TP29, TP290, TP291, TP292, TP293, TP294, TP295, TP296, TP297, TP298, TP299, TP3, TP30, TP300, TP301, TP302, TP303, TP304, TP305, TP306, TP307, TP308, TP309, TP31, TP310, TP311, TP312, TP32, TP33, TP34, TP35, TP36, TP37, TP38, TP39, TP4, TP40, TP41, TP42, TP43, TP44, TP45, TP46, TP47, TP48, TP49, TP5, TP50, TP51, TP52, TP53, TP54, TP55, TP56, TP57, TP58, TP59, TP6, TP60, TP61, TP62, TP63, TP64, TP65, TP66, TP67, TP68, TP69, TP7, TP70, TP71, TP72, TP73, TP74, TP75, TP76, TP77, TP78, TP79, TP8, TP80, TP81, TP82, TP83, TP84, TP85, TP86, TP87, TP88, TP89, TP9, TP90, TP91, TP92, TP93, TP94, TP95, TP96, TP97, TP98, TP99: TestPoint, symbol Connector:TestPoint
- added U10, U11, U12, U13, U14, U15, U16, U17, U18, U19, U20, U21, U22, U23, U24, U25, U26, U27, U28, U29, U30, U31, U4, U6, U8, U9: MPR121QR2, MPR121QR2:QFN40P300X300X60-20N, symbol MPR121QR2:MPR121QR2
- added U7: TCA9548APWR, PW24_TEX, symbol TCA9548APWR:TCA9548APWR
- J8: footprint marbastlib-various.pretty:USB_C_Receptacle_HRO_TYPE-C-31-M-12 -> USB:USB_C_Receptacle_HRO_TYPE-C-31-M-12; symbol Connector:USB_C_Receptacle_USB2.0_14P -> USB:USB_C_Receptacle_HRO_TYPE-C-31-M-12
- Q1: footprint symbols:SOT95P280X100-6N -> DMN3135LVT-7:DMN3135LVT-7
- S2, S3: footprint KEY-SMD_L3.0-W2.5-LS4.0 -> TS-1064S-A1B2-D4:TS-1064S-A1B2-D4; symbol Sensor PCB-altium-import:root_3_SW-PB_Miscellaneous Devices.IntLib -> TS-1064S-A1B2-D4:TS-1064S-A1B2-D4
- U3: footprint ESP32-WROOM-32E:ESP32-WROOM-32E -> RF_Module:ESP32-WROOM-32D
- U5: symbol Interface_USB:CH340C -> CH340C:CH340C
Connections:
- net +3.3V: now also C11.2, C13.2, C15.2, C25.2, C27.2, C29.2, C3.2, C31.2, C33.2, C35.2, C37.2, C39.2, C4.2, C41.2, C43.2, C45.2, C47.2, C49.2, C5.2, C53.2, C55.2, C57.2, C59.2, C6.2, C61.2, C9.2, R20.2, R21.2, R24.2, R25.2, R28.2, R29.2, R3.2, R30.2, R4.2, R5.2, U10.20 (VDD), U11.20 (VDD), U11.4 (ADDR), U12.20 (VDD), U13.20 (VDD), U14.20 (VDD), U15.20 (VDD), U15.4 (ADDR), U16.20 (VDD), U17.20 (VDD), U18.20 (VDD), U19.20 (VDD), U19.4 (ADDR), U20.20 (VDD), U21.20 (VDD), U22.20 (VDD), U23.20 (VDD), U23.4 (ADDR), U24.20 (VDD), U25.20 (VDD), U26.20 (VDD), U27.20 (VDD), U27.4 (ADDR), U28.20 (VDD), U29.20 (VDD), U30.20 (VDD), U31.20 (VDD), U31.4 (ADDR), U4.20 (VDD), U6.20 (VDD), U6.4 (ADDR), U7.24 (VCC), U8.20 (VDD), U9.20 (VDD)
- net GND: now also C1.2, C10.2, C11.1, C12.2, C13.1, C14.2, C15.1, C2.2, C24.2, C25.1, C26.2, C27.1, C28.2, C29.1, C3.1, C30.2, C31.1, C32.2, C33.1, C34.2, C35.1, C36.2, C37.1, C38.2, C39.1, C4.1, C40.2, C41.1, C42.2, C43.1, C44.2, C45.1, C46.2, C47.1, C48.2, C49.1, C5.1, C52.2, C53.1, C54.2, C55.1, C56.2, C57.1, C58.2, C59.1, C6.1, C60.2, C61.1, C62.2, C7.2, C8.2, C9.1, R22.2, R23.2, R26.2, R27.2, R31.2, R32.2, R33.2, R34.2, R35.2, R36.2, R37.2, R38.2, R39.2, R40.2, R41.2, R42.2, R43.2, R44.2, R45.2, R46.2, R47.2, R48.2, R49.2, R50.2, R51.2, R52.2, U10.4 (ADDR), U10.6 (VSS), U11.6 (VSS), U12.6 (VSS), U13.6 (VSS), U14.4 (ADDR), U14.6 (VSS), U15.6 (VSS), U16.6 (VSS), U17.6 (VSS), U18.4 (ADDR), U18.6 (VSS), U19.6 (VSS), U20.6 (VSS), U21.6 (VSS), U22.4 (ADDR), U22.6 (VSS), U23.6 (VSS), U24.6 (VSS), U25.6 (VSS), U26.4 (ADDR), U26.6 (VSS), U27.6 (VSS), U28.6 (VSS), U29.6 (VSS), U30.4 (ADDR), U30.6 (VSS), U31.6 (VSS), U4.4 (ADDR), U4.6 (VSS), U6.6 (VSS), U7.1 (A0), U7.12 (GND), U7.2 (A1), U7.21 (A2), U8.6 (VSS), U9.6 (VSS)
- net VB+: now also J2.1
- net VBo+: now also J2.2
- net IRQ5: now reaches U3.13 (IO14)
- net IRQ6: now reaches U3.16 (IO13)
- net SDA_IN: now reaches U3.33 (IO21)
- net SDA_IN: now also R4.1, U7.23 (SDA)
- net SCL_IN: now reaches U3.36 (IO22)
- net SCL_IN: now also R5.1, U7.22 (SCL)
- net CS renamed IRQ1
- net IRQ1: now also R21.1, U10.1 (~{IRQ}), U11.1 (~{IRQ}), U12.1 (~{IRQ}), U13.1 (~{IRQ})
- net DC renamed IRQ4
- net IRQ4: now also R28.1, R29.1, R30.1, U22.1 (~{IRQ}), U23.1 (~{IRQ}), U24.1 (~{IRQ}), U25.1 (~{IRQ}), U26.1 (~{IRQ}), U27.1 (~{IRQ}), U28.1 (~{IRQ}), U29.1 (~{IRQ}), U30.1 (~{IRQ}), U31.1 (~{IRQ})
- net L_Rst renamed IRQ0
- net IRQ0: now also R20.1, U4.1 (~{IRQ}), U6.1 (~{IRQ}), U8.1 (~{IRQ}), U9.1 (~{IRQ})
- net MOSI renamed IRQ2
- net IRQ2: now also R24.1, U14.1 (~{IRQ}), U15.1 (~{IRQ}), U16.1 (~{IRQ}), U17.1 (~{IRQ})
- net SCK renamed IRQ3
- net IRQ3: now also R25.1, U18.1 (~{IRQ}), U19.1 (~{IRQ}), U20.1 (~{IRQ}), U21.1 (~{IRQ})
- new net: C48.1, U25.5 (VREG)
- new net: TP187.1, U21.14 (ELEC6)
- new net: TP283.1, U29.14 (ELEC6)
- new net: TP143.1, U17.18 (ELEC10)
- new net: TP123.1, U16.10 (ELEC2)
- new net: TP49.1, U10.8 (ELEC0)
- new net: C38.1, U20.5 (VREG)
- new net: TP279.1, U29.10 (ELEC2)
- new net: TP280.1, U29.11 (ELEC3)
- new net: TP281.1, U29.12 (ELEC4)
- new net: TP282.1, U29.13 (ELEC5)
- new net: TP284.1, U29.15 (ELEC7)
- new net: TP285.1, U29.16 (ELEC8)
- new net: TP286.1, U29.17 (ELEC9)
- new net: TP287.1, U29.18 (ELEC10)
- new net: TP288.1, U29.19 (ELEC11)
- new net: C58.1, U29.5 (VREG)
- new net: R50.1, U29.7 (REXT)
- new net: TP277.1, U29.8 (ELEC0)
- new net: TP278.1, U29.9 (ELEC1)
- new net: TP246.1, U26.13 (ELEC5)
- new net: TP46.1, U9.17 (ELEC9)
- new net: TP197.1, U22.12 (ELEC4)
- new net: TP29.1, U8.12 (ELEC4)
- new net: TP222.1, U24.13 (ELEC5)
- new net: TP247.1, U26.14 (ELEC6)
- new net: TP110.1, U15.9 (ELEC1)
- new net: TP276.1, U28.19 (ELEC11)
- new net: TP122.1, U16.9 (ELEC1)
- new net: TP249.1, U26.16 (ELEC8)
- new net: TP205.1, U23.8 (ELEC0)
- new net: TP18.1, U6.13 (ELEC5)
- new net: TP92.1, U13.15 (ELEC7)
- new net: TP40.1, U9.11 (ELEC3)
- new net: C30.1, U16.5 (VREG)
- new net: TP161.1, U19.12 (ELEC4)
- new net: C12.1, U11.5 (VREG)
- new net: TP309.1, U31.16 (ELEC8)
- new net: TP65.1, U11.12 (ELEC4)
- new net: TP265.1, U28.8 (ELEC0)
- new net: TP31.1, U8.14 (ELEC6)
- new net: TP235.1, U25.14 (ELEC6)
- new net: TP275.1, U28.18 (ELEC10)
- new net: TP24.1, U6.19 (ELEC11)
- new net: TP252.1, U26.19 (ELEC11)
- new net: TP55.1, U10.14 (ELEC6)
- new net: TP98.1, U14.9 (ELEC1)
- new net: R42.1, U21.7 (REXT)
- new net: TP231.1, U25.10 (ELEC2)
- new net: TP232.1, U25.11 (ELEC3)
- new net: TP233.1, U25.12 (ELEC4)
- new net: TP234.1, U25.13 (ELEC5)
- new net: TP236.1, U25.15 (ELEC7)
- new net: TP237.1, U25.16 (ELEC8)
- new net: TP238.1, U25.17 (ELEC9)
- new net: TP239.1, U25.18 (ELEC10)
- new net: TP240.1, U25.19 (ELEC11)
- new net: R46.1, U25.7 (REXT)
- new net: TP229.1, U25.8 (ELEC0)
- new net: TP230.1, U25.9 (ELEC1)
- new net: TP109.1, U15.8 (ELEC0)
- new net: TP185.1, U21.12 (ELEC4)
- new net: TP135.1, U17.10 (ELEC2)
- new net: TP136.1, U17.11 (ELEC3)
- new net: TP75.1, U12.10 (ELEC2)
- new net: TP76.1, U12.11 (ELEC3)
- new net: TP77.1, U12.12 (ELEC4)
- new net: TP78.1, U12.13 (ELEC5)
- new net: TP79.1, U12.14 (ELEC6)
- new net: TP80.1, U12.15 (ELEC7)
- new net: TP81.1, U12.16 (ELEC8)
- new net: TP82.1, U12.17 (ELEC9)
- new net: TP83.1, U12.18 (ELEC10)
- new net: TP84.1, U12.19 (ELEC11)
- new net: C14.1, U12.5 (VREG)
- new net: R33.1, U12.7 (REXT)
- new net: TP73.1, U12.8 (ELEC0)
- new net: TP74.1, U12.9 (ELEC1)
- new net: TP114.1, U15.13 (ELEC5)
- new net: C40.1, U21.5 (VREG)
- new net: TP244.1, U26.11 (ELEC3)
- new net: TP190.1, U21.17 (ELEC9)
- new net: TP12.1, U4.19 (ELEC11)
- new net: TP147.1, U18.10 (ELEC2)
- new net: TP225.1, U24.16 (ELEC8)
- new net: TP296.1, U30.15 (ELEC7)
- new net: TP104.1, U14.15 (ELEC7)
- new net: TP35.1, U8.18 (ELEC10)
- new net: TP180.1, U20.19 (ELEC11)
- new net: C54.1, U27.5 (VREG)
- new net: TP208.1, U23.11 (ELEC3)
- new net: TP151.1, U18.14 (ELEC6)
- new net: TP291.1, U30.10 (ELEC2)
- new net: TP292.1, U30.11 (ELEC3)
- new net: TP293.1, U30.12 (ELEC4)
- new net: TP294.1, U30.13 (ELEC5)
- new net: TP295.1, U30.14 (ELEC6)
- new net: TP297.1, U30.16 (ELEC8)
- new net: TP298.1, U30.17 (ELEC9)
- new net: TP299.1, U30.18 (ELEC10)
- new net: TP300.1, U30.19 (ELEC11)
- new net: C60.1, U30.5 (VREG)
- new net: R51.1, U30.7 (REXT)
- new net: TP289.1, U30.8 (ELEC0)
- new net: TP290.1, U30.9 (ELEC1)
- new net: R27.1, U9.7 (REXT)
- new net: TP206.1, U23.9 (ELEC1)
- new net: TP87.1, U13.10 (ELEC2)
- new net: TP88.1, U13.11 (ELEC3)
- new net: TP89.1, U13.12 (ELEC4)
- new net: TP90.1, U13.13 (ELEC5)
- new net: TP91.1, U13.14 (ELEC6)
- new net: TP93.1, U13.16 (ELEC8)
- new net: TP94.1, U13.17 (ELEC9)
- new net: TP95.1, U13.18 (ELEC10)
- new net: TP96.1, U13.19 (ELEC11)
- new net: C24.1, U13.5 (VREG)
- new net: R34.1, U13.7 (REXT)
- new net: TP85.1, U13.8 (ELEC0)
- new net: TP86.1, U13.9 (ELEC1)
- new net: TP156.1, U18.19 (ELEC11)
- new net: TP159.1, U19.10 (ELEC2)
- new net: TP160.1, U19.11 (ELEC3)
- new net: TP162.1, U19.13 (ELEC5)
- new net: TP163.1, U19.14 (ELEC6)
- new net: TP164.1, U19.15 (ELEC7)
- new net: TP165.1, U19.16 (ELEC8)
- new net: TP166.1, U19.17 (ELEC9)
- new net: TP167.1, U19.18 (ELEC10)
- new net: TP168.1, U19.19 (ELEC11)
- new net: C36.1, U19.5 (VREG)
- new net: R40.1, U19.7 (REXT)
- new net: TP157.1, U19.8 (ELEC0)
- new net: TP158.1, U19.9 (ELEC1)
- new net: C56.1, U28.5 (VREG)
- new net: TP142.1, U17.17 (ELEC9)
- new net: TP62.1, U11.9 (ELEC1)
- new net: TP140.1, U17.15 (ELEC7)
- new net: TP118.1, U15.17 (ELEC9)
- new net: R35.1, U14.7 (REXT)
- new net: TP170.1, U20.9 (ELEC1)
- new net: R36.1, U15.7 (REXT)
- new net: TP99.1, U14.10 (ELEC2)
- new net: R43.1, U22.7 (REXT)
- new net: TP242.1, U26.9 (ELEC1)
- new net: C8.1, U9.5 (VREG)
- new net: TP2.1, U4.9 (ELEC1)
- new net: TP312.1, U31.19 (ELEC11)
- new net: TP195.1, U22.10 (ELEC2)
- new net: TP196.1, U22.11 (ELEC3)
- new net: TP198.1, U22.13 (ELEC5)
- new net: TP199.1, U22.14 (ELEC6)
- new net: TP200.1, U22.15 (ELEC7)
- new net: TP201.1, U22.16 (ELEC8)
- new net: TP202.1, U22.17 (ELEC9)
- new net: TP203.1, U22.18 (ELEC10)
- new net: TP204.1, U22.19 (ELEC11)
- new net: C42.1, U22.5 (VREG)
- new net: TP193.1, U22.8 (ELEC0)
- new net: TP194.1, U22.9 (ELEC1)
- new net: TP243.1, U26.10 (ELEC2)
- new net: TP245.1, U26.12 (ELEC4)
- new net: TP248.1, U26.15 (ELEC7)
- new net: TP250.1, U26.17 (ELEC9)
- new net: TP251.1, U26.18 (ELEC10)
- new net: C52.1, U26.5 (VREG)
- new net: R47.1, U26.7 (REXT)
- new net: TP241.1, U26.8 (ELEC0)
- new net: TP1.1, U4.8 (ELEC0)
- new net: TP8.1, U4.15 (ELEC7)
- new net: TP132.1, U16.19 (ELEC11)
- new net: TP66.1, U11.13 (ELEC5)
- new net: TP27.1, U8.10 (ELEC2)
- new net: TP28.1, U8.11 (ELEC3)
- new net: TP30.1, U8.13 (ELEC5)
- new net: TP32.1, U8.15 (ELEC7)
- new net: TP33.1, U8.16 (ELEC8)
- new net: TP34.1, U8.17 (ELEC9)
- new net: TP36.1, U8.19 (ELEC11)
- new net: C7.1, U8.5 (VREG)
- new net: R26.1, U8.7 (REXT)
- new net: TP25.1, U8.8 (ELEC0)
- new net: TP26.1, U8.9 (ELEC1)
- new net: TP260.1, U27.15 (ELEC7)
- new net: TP183.1, U21.10 (ELEC2)
- new net: TP184.1, U21.11 (ELEC3)
- new net: TP186.1, U21.13 (ELEC5)
- new net: TP188.1, U21.15 (ELEC7)
- new net: TP189.1, U21.16 (ELEC8)
- new net: TP191.1, U21.18 (ELEC10)
- new net: TP192.1, U21.19 (ELEC11)
- new net: TP181.1, U21.8 (ELEC0)
- new net: TP182.1, U21.9 (ELEC1)
- new net: TP267.1, U28.10 (ELEC2)
- new net: TP269.1, U28.12 (ELEC4)
- new net: R32.1, U11.7 (REXT)
- new net: TP215.1, U23.18 (ELEC10)
- new net: TP219.1, U24.10 (ELEC2)
- new net: TP218.1, U24.9 (ELEC1)
- new net: TP11.1, U4.18 (ELEC10)
- new net: TP145.1, U18.8 (ELEC0)
- new net: TP211.1, U23.14 (ELEC6)
- new net: R22.1, U4.7 (REXT)
- new net: R38.1, U17.7 (REXT)
- new net: TP113.1, U15.12 (ELEC4)
- new net: TP44.1, U9.15 (ELEC7)
- new net: R45.1, U24.7 (REXT)
- new net: TP67.1, U11.14 (ELEC6)
- new net: TP172.1, U20.11 (ELEC3)
- new net: TP39.1, U9.10 (ELEC2)
- new net: TP60.1, U10.19 (ELEC11)
- new net: C26.1, U14.5 (VREG)
- new net: TP209.1, U23.12 (ELEC4)
- new net: TP257.1, U27.12 (ELEC4)
- new net: TP307.1, U31.14 (ELEC6)
- new net: TP120.1, U15.19 (ELEC11)
- new net: TP101.1, U14.12 (ELEC4)
- new net: TP50.1, U10.9 (ELEC1)
- new net: TP130.1, U16.17 (ELEC9)
- new net: TP213.1, U23.16 (ELEC8)
- new net: TP272.1, U28.15 (ELEC7)
- new net: R41.1, U20.7 (REXT)
- new net: TP148.1, U18.11 (ELEC3)
- new net: TP174.1, U20.13 (ELEC5)
- new net: TP311.1, U31.18 (ELEC10)
- new net: TP48.1, U9.19 (ELEC11)
- new net: TP7.1, U4.14 (ELEC6)
- new net: TP100.1, U14.11 (ELEC3)
- new net: TP220.1, U24.11 (ELEC3)
- new net: TP221.1, U24.12 (ELEC4)
- new net: TP223.1, U24.14 (ELEC6)
- new net: TP224.1, U24.15 (ELEC7)
- new net: TP226.1, U24.17 (ELEC9)
- new net: TP227.1, U24.18 (ELEC10)
- new net: TP228.1, U24.19 (ELEC11)
- new net: C46.1, U24.5 (VREG)
- new net: TP217.1, U24.8 (ELEC0)
- new net: R49.1, U28.7 (REXT)
- new net: TP305.1, U31.12 (ELEC4)
- new net: TP16.1, U6.11 (ELEC3)
- new net: TP47.1, U9.18 (ELEC10)
- new net: TP117.1, U15.16 (ELEC8)
- new net: TP258.1, U27.13 (ELEC5)
- new net: R37.1, U16.7 (REXT)
- new net: TP119.1, U15.18 (ELEC10)
- new net: TP64.1, U11.11 (ELEC3)
- new net: TP106.1, U14.17 (ELEC9)
- new net: TP179.1, U20.18 (ELEC10)
- new net: TP68.1, U11.15 (ELEC7)
- new net: C1.1, U4.5 (VREG)
- new net: TP210.1, U23.13 (ELEC5)
- new net: TP253.1, U27.8 (ELEC0)
- new net: TP19.1, U6.14 (ELEC6)
- new net: TP310.1, U31.17 (ELEC9)
- new net: TP149.1, U18.12 (ELEC4)
- new net: TP150.1, U18.13 (ELEC5)
- new net: TP152.1, U18.15 (ELEC7)
- new net: TP153.1, U18.16 (ELEC8)
- new net: TP154.1, U18.17 (ELEC9)
- new net: TP155.1, U18.18 (ELEC10)
- new net: C34.1, U18.5 (VREG)
- new net: R39.1, U18.7 (REXT)
- new net: TP146.1, U18.9 (ELEC1)
- new net: TP17.1, U6.12 (ELEC4)
- new net: TP255.1, U27.10 (ELEC2)
- new net: R23.1, U6.7 (REXT)
- new net: TP131.1, U16.18 (ELEC10)
- new net: TP22.1, U6.17 (ELEC9)
- new net: TP137.1, U17.12 (ELEC4)
- new net: TP138.1, U17.13 (ELEC5)
- new net: TP139.1, U17.14 (ELEC6)
- new net: TP141.1, U17.16 (ELEC8)
- new net: TP144.1, U17.19 (ELEC11)
- new net: C32.1, U17.5 (VREG)
- new net: TP133.1, U17.8 (ELEC0)
- new net: TP134.1, U17.9 (ELEC1)
- new net: TP176.1, U20.15 (ELEC7)
- new net: TP175.1, U20.14 (ELEC6)
- new net: TP38.1, U9.9 (ELEC1)
- new net: TP125.1, U16.12 (ELEC4)
- new net: TP107.1, U14.18 (ELEC10)
- new net: TP53.1, U10.12 (ELEC4)
- new net: TP254.1, U27.9 (ELEC1)
- new net: TP173.1, U20.12 (ELEC4)
- new net: TP256.1, U27.11 (ELEC3)
- new net: TP259.1, U27.14 (ELEC6)
- new net: TP261.1, U27.16 (ELEC8)
- new net: TP262.1, U27.17 (ELEC9)
- new net: TP263.1, U27.18 (ELEC10)
- new net: TP264.1, U27.19 (ELEC11)
- new net: R48.1, U27.7 (REXT)
- new net: TP128.1, U16.15 (ELEC7)
- new net: TP51.1, U10.10 (ELEC2)
- new net: TP52.1, U10.11 (ELEC3)
- new net: TP54.1, U10.13 (ELEC5)
- new net: TP56.1, U10.15 (ELEC7)
- new net: TP57.1, U10.16 (ELEC8)
- new net: TP58.1, U10.17 (ELEC9)
- new net: TP59.1, U10.18 (ELEC10)
- new net: C10.1, U10.5 (VREG)
- new net: R31.1, U10.7 (REXT)
- new net: TP268.1, U28.11 (ELEC3)
- new net: TP5.1, U4.12 (ELEC4)
- new net: TP216.1, U23.19 (ELEC11)
- new net: TP21.1, U6.16 (ELEC8)
- new net: TP69.1, U11.16 (ELEC8)
- new net: TP6.1, U4.13 (ELEC5)
- new net: TP63.1, U11.10 (ELEC2)
- new net: C62.1, U31.5 (VREG)
- new net: C28.1, U15.5 (VREG)
- new net: TP207.1, U23.10 (ELEC2)
- new net: TP212.1, U23.15 (ELEC7)
- new net: TP214.1, U23.17 (ELEC9)
- new net: C44.1, U23.5 (VREG)
- new net: R44.1, U23.7 (REXT)
- new net: TP116.1, U15.15 (ELEC7)
- new net: TP41.1, U9.12 (ELEC4)
- new net: TP42.1, U9.13 (ELEC5)
- new net: TP43.1, U9.14 (ELEC6)
- new net: TP45.1, U9.16 (ELEC8)
- new net: TP37.1, U9.8 (ELEC0)
- new net: TP121.1, U16.8 (ELEC0)
- new net: TP72.1, U11.19 (ELEC11)
- new net: TP303.1, U31.10 (ELEC2)
- new net: TP304.1, U31.11 (ELEC3)
- new net: TP306.1, U31.13 (ELEC5)
- new net: TP308.1, U31.15 (ELEC7)
- new net: R52.1, U31.7 (REXT)
- new net: TP301.1, U31.8 (ELEC0)
- new net: TP302.1, U31.9 (ELEC1)
- new net: TP111.1, U15.10 (ELEC2)
- new net: TP112.1, U15.11 (ELEC3)
- new net: TP115.1, U15.14 (ELEC6)
- new net: TP126.1, U16.13 (ELEC5)
- new net: TP105.1, U14.16 (ELEC8)
- new net: TP3.1, U4.10 (ELEC2)
- new net: TP4.1, U4.11 (ELEC3)
- new net: TP9.1, U4.16 (ELEC8)
- new net: TP10.1, U4.17 (ELEC9)
- new net: TP71.1, U11.18 (ELEC10)
- new net: TP169.1, U20.8 (ELEC0)
- new net: TP103.1, U14.14 (ELEC6)
- new net: C2.1, U6.5 (VREG)
- new net: TP129.1, U16.16 (ELEC8)
- new net: TP70.1, U11.17 (ELEC9)
- new net: TP61.1, U11.8 (ELEC0)
- new net: TP266.1, U28.9 (ELEC1)
- new net: TP102.1, U14.13 (ELEC5)
- new net: TP178.1, U20.17 (ELEC9)
- new net: TP274.1, U28.17 (ELEC9)
- new net: TP124.1, U16.11 (ELEC3)
- new net: TP127.1, U16.14 (ELEC6)
- new net: TP15.1, U6.10 (ELEC2)
- new net: TP177.1, U20.16 (ELEC8)
- new net: TP20.1, U6.15 (ELEC7)
- new net: TP23.1, U6.18 (ELEC10)
- new net: TP13.1, U6.8 (ELEC0)
- new net: TP14.1, U6.9 (ELEC1)
- new net: TP270.1, U28.13 (ELEC5)
- new net: TP271.1, U28.14 (ELEC6)
- new net: TP273.1, U28.16 (ELEC8)
- new net: TP171.1, U20.10 (ELEC2)
- new net: TP97.1, U14.8 (ELEC0)
- new net: TP108.1, U14.19 (ELEC11)
- new net I2C_RESET_IN: R3.1, U7.3 (*RESET)
- new net SCA6: U7.18 (SC6)
- new net SCL0: U4.2 (SCL), U6.2 (SCL), U7.5 (SC0), U8.2 (SCL), U9.2 (SCL), U9.4 (ADDR)
- new net SCL1: U10.2 (SCL), U11.2 (SCL), U12.2 (SCL), U13.2 (SCL), U13.4 (ADDR), U7.7 (SC1)
- new net SCL2: U14.2 (SCL), U15.2 (SCL), U16.2 (SCL), U17.2 (SCL), U17.4 (ADDR), U7.9 (SC2)
- new net SCL3: U18.2 (SCL), U19.2 (SCL), U20.2 (SCL), U21.2 (SCL), U21.4 (ADDR), U7.11 (SC3)
- new net SCL4: U22.2 (SCL), U23.2 (SCL), U24.2 (SCL), U25.2 (SCL), U25.4 (ADDR), U7.14 (SC4)
- new net SCL5: U26.2 (SCL), U27.2 (SCL), U28.2 (SCL), U29.2 (SCL), U29.4 (ADDR), U7.16 (SC5)
- new net SCL6: U30.2 (SCL), U31.2 (SCL)
- new net SCL7: U7.20 (SC7)
- new net SDA0: U4.3 (SDA), U6.3 (SDA), U7.4 (SD0), U8.3 (SDA), U8.4 (ADDR), U9.3 (SDA)
- new net SDA1: U10.3 (SDA), U11.3 (SDA), U12.3 (SDA), U12.4 (ADDR), U13.3 (SDA), U7.6 (SD1)
- new net SDA2: U14.3 (SDA), U15.3 (SDA), U16.3 (SDA), U16.4 (ADDR), U17.3 (SDA), U7.8 (SD2)
- new net SDA3: U18.3 (SDA), U19.3 (SDA), U20.3 (SDA), U20.4 (ADDR), U21.3 (SDA), U7.10 (SD3)
- new net SDA4: U22.3 (SDA), U23.3 (SDA), U24.3 (SDA), U24.4 (ADDR), U25.3 (SDA), U7.13 (SD4)
- new net SDA5: U26.3 (SDA), U27.3 (SDA), U28.3 (SDA), U28.4 (ADDR), U29.3 (SDA)
- new net SDA6: U30.3 (SDA), U31.3 (SDA), U7.17 (SD6)
- new net SDA7: U7.19 (SD7)
- new net SDL5: U7.15 (SD5)
Other:
- note added: "A#0 Key"
- note added: "A0 Key"
- note added: "B0 Key"
- note added: "C#0 Key"
- note added: "C0 Key"
- note added: "C1 Key"
- note added: "D#0 Key"
- note added: "D0 Key"
- note added: "E0 Key"
- note added: "F#0 Key"
- note added: "F0 Key"
- note added: "G#0 Key"
- note added: "G0 Key"
- note added: "I2C Multiplexer"
- note added: "IRQ0"
- note added: "IRQ1"
- note added: "IRQ2"
- note added: "IRQ3"
- note added: "IRQ4"
- note added: "IRQ5"
- note added: "IRQ6"
- note added: "USB"
- note removed: "LCD"
- moved on the sheet: C16, C17, C18, C19, C20, C21, C22, C23, C50, C51, D1, D2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

Commit message: Update embedded keyboard schematic for 12 segments
Parts:
- removed C35, C36, C37, C38, C39, C40, C41, C42, C43, C44, C45, C46, C47, C48, C49, C52, C53, C54, C55, C56, C57, C58, C59, C60, C61, C62: 100nF, CAP_CL03_SAM, symbol CL03A104KP3NNNC:CL03A104KP3NNNC
- removed R25, R29: 10K, Resistor_SMD:R_0402_1005Metric, symbol Device:R
- removed R26, R32, R34, R36, R38, R40, R42, R44, R46, R47, R48, R49, R50, R51, R52: 75K, RT0805FRE0775KL:RESC2012X60N, symbol RT0805FRE0775KL:RT0805FRE0775KL
- removed TP157, TP158, TP159, TP160, TP161, TP162, TP163, TP164, TP165, TP166, TP167, TP168, TP169, TP170, TP171, TP172, TP173, TP174, TP175, TP176, TP177, TP178, TP179, TP180, TP181, TP182, TP183, TP184, TP185, TP186, TP187, TP188, TP189, TP190, TP191, TP192, TP193, TP194, TP195, TP196, TP197, TP198, TP199, TP200, TP201, TP202, TP203, TP204, TP205, TP206, TP207, TP208, TP209, TP210, TP211, TP212, TP213, TP214, TP215, TP216, TP217, TP218, TP219, TP220, TP221, TP222, TP223, TP224, TP225, TP226, TP227, TP228, TP229, TP230, TP231, TP232, TP233, TP234, TP235, TP236, TP237, TP238, TP239, TP240, TP241, TP242, TP243, TP244, TP245, TP246, TP247, TP248, TP249, TP250, TP251, TP252, TP253, TP254, TP255, TP256, TP257, TP258, TP259, TP260, TP261, TP262, TP263, TP264, TP265, TP266, TP267, TP268, TP269, TP270, TP271, TP272, TP273, TP274, TP275, TP276, TP277, TP278, TP279, TP280, TP281, TP282, TP283, TP284, TP285, TP286, TP287, TP288, TP289, TP290, TP291, TP292, TP293, TP294, TP295, TP296, TP297, TP298, TP299, TP300, TP301, TP302, TP303, TP304, TP305, TP306, TP307, TP308, TP309, TP310, TP311, TP312: TestPoint, symbol Connector:TestPoint
- removed U19, U20, U21, U22, U23, U24, U25, U26, U27, U28, U29, U30, U31, U6: MPR121QR2, MPR121QR2:QFN40P300X300X60-20N, symbol MPR121QR2:MPR121QR2
- added R25, R29: 75K, RT0805FRE0775KL:RESC2012X60N, symbol RT0805FRE0775KL:RT0805FRE0775KL
- added R26, R32, R34, R36, R38, R40, R42, R44: 10K, Resistor_SMD:R_0402_1005Metric, symbol Device:R
- added U7: MPR121QR2, MPR121QR2:QFN40P300X300X60-20N, symbol MPR121QR2:MPR121QR2
- renumbered U5 to U4, U7 to U5, U4 to U6
Connections:
- net +3.3V: now also C2.2, C7.2, R26.2, R32.2, R34.2, R36.2, R38.2, R40.2, R42.2, R44.2, U7.20 (VDD); no longer C4.2, C6.2, U11.4 (ADDR), U15.4 (ADDR)
- net GND: now also C2.1, C4.2, C6.2, C7.1, U11.4 (ADDR), U12.4 (ADDR), U13.4 (ADDR), U15.4 (ADDR), U16.4 (ADDR), U17.4 (ADDR), U8.4 (ADDR), U9.4 (ADDR), R25.2, R29.2, U7.4 (ADDR), U7.6 (VSS); no longer C2.2, C4.1, C6.1, C7.2
- net IRQ0: no longer U8.1 (~{IRQ}), U9.1 (~{IRQ})
- net IRQ1: now also U7.1 (~{IRQ}); no longer U10.1 (~{IRQ}), U11.1 (~{IRQ}), U12.1 (~{IRQ}), U13.1 (~{IRQ})
- net IRQ2: now also U8.1 (~{IRQ}); no longer U14.1 (~{IRQ}), U15.1 (~{IRQ}), U16.1 (~{IRQ}), U17.1 (~{IRQ})
- net IRQ3: now also U9.1 (~{IRQ}), R26.1; no longer U18.1 (~{IRQ})
- net IRQ4: now also U10.1 (~{IRQ}); no longer R30.1
- net IRQ5: now also R30.1, U11.1 (~{IRQ})
- net IRQ6: now also U12.1 (~{IRQ}), R32.1
- net SCL0: now also U7.2 (SCL); no longer U8.2 (SCL), U9.2 (SCL), U9.4 (ADDR)
- net SCL1: now also U8.2 (SCL), U9.2 (SCL); no longer U10.2 (SCL), U11.2 (SCL), U12.2 (SCL), U13.2 (SCL), U13.4 (ADDR)
- net SCL2: now also U10.2 (SCL), U11.2 (SCL); no longer U14.2 (SCL), U15.2 (SCL), U16.2 (SCL), U17.2 (SCL), U17.4 (ADDR)
- net SCL3: now also U12.2 (SCL), U13.2 (SCL); no longer U18.2 (SCL)
- net SCL4: now also U14.2 (SCL), U15.2 (SCL)
- net SCL5: now also U16.2 (SCL), U17.2 (SCL)
- net SCL6: now also U18.2 (SCL)
- net SDA0: now also U7.3 (SDA); no longer U8.3 (SDA), U8.4 (ADDR), U9.3 (SDA)
- net SDA1: now also U8.3 (SDA), U9.3 (SDA); no longer U10.3 (SDA), U11.3 (SDA), U12.3 (SDA), U12.4 (ADDR), U13.3 (SDA)
- net SDA2: now also U10.3 (SDA), U11.3 (SDA); no longer U14.3 (SDA), U15.3 (SDA), U16.3 (SDA), U16.4 (ADDR), U17.3 (SDA)
- net SDA3: now also U12.3 (SDA), U13.3 (SDA); no longer U18.3 (SDA)
- net SDA4: now also U14.3 (SDA), U15.3 (SDA)
- net SDA5: now also U16.3 (SDA), U17.3 (SDA)
- net SDA6: now also U18.3 (SDA)
- net at TP18.1: now also U7.13 (ELEC5)
- net at TP24.1: now also U7.19 (ELEC11)
- net at U13.7 (REXT): now also R35.1
- net at U14.7 (REXT): now also R37.1; no longer R35.1
- net at U15.7 (REXT): now also R39.1
- net at R43.1: now also U17.7 (REXT)
- net at U8.5 (VREG): now also C6.1; no longer C7.1
- net at U8.7 (REXT): now also R25.1
- net at U11.7 (REXT): now also R31.1
- net at R45.1: now also U18.7 (REXT)
- net at R41.1: now also U16.7 (REXT)
- net at TP16.1: now also U7.11 (ELEC3)
- net at TP19.1: now also U7.14 (ELEC6)
- net at TP17.1: now also U7.12 (ELEC4)
- net at R23.1: now also U7.7 (REXT)
- net at TP22.1: now also U7.17 (ELEC9)
- net at U10.7 (REXT): now also R29.1; no longer R31.1
- net at TP21.1: now also U7.16 (ELEC8)
- net IRQ9: now reaches U3.27 (IO16)
- net IRQ9: now also U15.1 (~{IRQ}), R38.1
- net IRQ10: now reaches U3.28 (IO17)
- net IRQ10: now also U16.1 (~{IRQ}), R40.1
- net IRQ11: now reaches U3.30 (IO18)
- net IRQ11: now also U17.1 (~{IRQ}), R42.1
- net IRQ12: now reaches U3.31 (IO19)
- net IRQ12: now also U18.1 (~{IRQ}), R44.1
- net IRQ7: now reaches U3.6 (IO34)
- net IRQ7: now also U13.1 (~{IRQ}), R34.1
- net IRQ8: now reaches U3.7 (IO35)
- net IRQ8: now also U14.1 (~{IRQ}), R36.1
- net at TP15.1: now also U7.10 (ELEC2)
- net at TP20.1: now also U7.15 (ELEC7)
- net at TP23.1: now also U7.18 (ELEC10)
- net at TP13.1: now also U7.8 (ELEC0)
- net at TP14.1: now also U7.9 (ELEC1)
- new net: C4.1, U7.5 (VREG)
Other:
- note removed: "IRQ0"
- note removed: "IRQ1"
- note removed: "IRQ2"
- note removed: "IRQ3"
- note removed: "IRQ4"
- note removed: "IRQ5"
- note removed: "IRQ6"
- company: (none) -> 01 Binary
- title: (none) -> Embedded Keyboard
- moved on the sheet: C1, C3, H1, H2, H3, H4, H5, H6, H7, R20, R22, TP1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

Commit message: Final pre-submission
Parts:
- C1, C10, C11, C12, C13, C14, C15, C2, C24, C25, C26, C27, C28, C29, C3, C30, C31, C32, C33, C34, C4, C5, C6, C7, C8, C9: footprint CAP_CL03_SAM -> CL03A104KP3NNNC:CL03A104KP3NNNC
- C16, C22, C50, C51: footprint Capacitor_SMD:C_0402_1005Metric -> CL03A104KP3NNNC:CL03A104KP3NNNC
- C17, C18, C23: footprint Capacitor_Tantalum_SMD:CP_EIA-3216-10_Kemet-I -> CC0805KKX5R5BB106:CC0805KKX5R5BB106
- C19, C20, C21: footprint Capacitor_SMD:C_0402_1005Metric -> CC0805KKX5R5BB106:CC0805KKX5R5BB106
- D1: footprint LED_SMD:LED_0603_1608Metric -> 150080GS75000:150080GS75000
- D2: footprint LED_SMD:LED_0603_1608Metric -> 150080SS75000:150080SS75000
- H1, H2, H3, H4, H5, H6, H7: footprint (none) -> MountingHole:MountingHole_2.2mm_M2_Pad
- R1, R2: footprint Resistor_SMD:R_0402_1005Metric -> 0402WGF5101TCE:0402WGF5101TCE
- R10: footprint Resistor_SMD:R_0402_1005Metric -> RC0805FR-07100KL:RC0805FR-07100KL
- R11: footprint Resistor_SMD:R_0402_1005Metric -> RC0805FR-072K49L:RC0805FR-072K49L
- R12, R14, R15, R16, R20, R21, R24, R26, R28, R3, R30, R32, R34, R36, R38, R4, R40, R42, R44, R5, R6, R7, R8, R9: footprint Resistor_SMD:R_0402_1005Metric -> AF0805FR-0710KL:AF0805FR-0710KL
- R13, R19: footprint Resistor_SMD:R_0402_1005Metric -> RE0805FRE071KL:RE0805FRE071KL
- R17, R18: footprint Resistor_SMD:R_0402_1005Metric -> RTT01513JTH:RTT01513JTH
- R22, R23, R25, R27, R29, R31, R33, R35, R37, R39, R41, R43, R45: footprint RT0805FRE0775KL:RESC2012X60N -> RT0805FRE0775KL:RT0805FRE0775KL
- U1: footprint LM3671MFX-3.3_NOPB:LM3671MFX-3.3_NOPB -> CC0805KKX5R5BB106:CC0805KKX5R5BB106
- U10, U11, U12, U13, U14, U15, U16, U17, U18, U6, U7, U8, U9: footprint MPR121QR2:QFN40P300X300X60-20N -> MPR121QR2:MPR121QR2
- U3: footprint RF_Module:ESP32-WROOM-32D -> ESP32-WROOM-32E-N4:ESP32-WROOM-32E-N4
- U4: footprint Package_SO:SOIC-16_3.9x9.9mm_P1.27mm -> CH340C:CH340C
- U5: footprint PW24_TEX -> MCP73831T-2ACI-OT:MCP73831T-2ACI-OT
Connections:
- no-connect marks 0 -> 10

Commit message: Re-designed keyboard
Parts:
- C1, C10, C11, C12, C13, C14, C15, C2, C24, C25, C26, C27, C28, C29, C3, C30, C31, C32, C33, C34, C4, C5, C6, C7, C8, C9: footprint CL03A104KP3NNNC:CL03A104KP3NNNC -> Capacitor_SMD:C_0402_1005Metric; LCSC Part Number (none) -> C1525
- C16, C22: footprint CL03A104KP3NNNC:CL03A104KP3NNNC -> Capacitor_SMD:C_0402_1005Metric; LCSC Part no C49062 -> (none)
- C17, C18, C23: footprint CC0805KKX5R5BB106:CC0805KKX5R5BB106 -> Capacitor_Tantalum_SMD:CP_EIA-3216-18_Kemet-A; LCSC Part no C7171 -> (none)
- C19, C20, C21: footprint CC0805KKX5R5BB106:CC0805KKX5R5BB106 -> Capacitor_SMD:C_0402_1005Metric; LCSC Part no C49062 -> (none)
- C50, C51: footprint CL03A104KP3NNNC:CL03A104KP3NNNC -> Capacitor_SMD:C_0402_1005Metric
- J1, J2: LCSC Part Number C295747 -> C51940124
- Q1: LCSC Part no C155326 -> (none)
- R1, R2: footprint 0402WGF5101TCE:0402WGF5101TCE -> Resistor_SMD:R_0402_1005Metric
- R10: footprint RC0805FR-07100KL:RC0805FR-07100KL -> Resistor_SMD:R_0402_1005Metric; LCSC Part no C100126 -> (none)
- R11: footprint RC0805FR-072K49L:RC0805FR-072K49L -> Resistor_SMD:R_0402_1005Metric; LCSC Part no C100126 -> (none)
- R12, R14, R15, R16, R20, R21, R24, R26, R28, R3, R30, R32, R34, R36, R38, R4, R40, R42, R44, R5, R6, R9: footprint AF0805FR-0710KL:AF0805FR-0710KL -> Resistor_SMD:R_0402_1005Metric; LCSC Part no C100126 -> (none)
- R13, R19: footprint RE0805FRE071KL:RE0805FRE071KL -> Resistor_SMD:R_0402_1005Metric; LCSC Part no C100126 -> (none)
- R17, R18: footprint RTT01513JTH:RTT01513JTH -> Resistor_SMD:R_0402_1005Metric; LCSC Part no C102736 -> (none)
- R22, R23, R25, R27, R29, R31, R33, R35, R37, R39, R41, R43, R45: footprint RT0805FRE0775KL:RT0805FRE0775KL -> Resistor_SMD:R_0402_1005Metric; LCSC Part Number (none) -> C25798
- R7, R8: value 10K -> 22R; footprint AF0805FR-0710KL:AF0805FR-0710KL -> Resistor_SMD:R_0402_1005Metric; LCSC Part Number C25744 -> C17561; LCSC Part no C100126 -> (none)
- U1: footprint CC0805KKX5R5BB106:CC0805KKX5R5BB106 -> SSW:SOT95P280X145-5N
- U10, U11, U12, U13, U14, U15, U16, U17, U18, U6, U7, U8, U9: LCSC Part Number (none) -> C91322
- U3: LCSC Part Number C701341 -> C328062
- U4: LCSC Part no C7464026 -> (none)
- U5: footprint MCP73831T-2ACI-OT:MCP73831T-2ACI-OT -> symbols:SOP65P640X120-24N; LCSC Part Number (none) -> C130026
Connections:
- net SCA6 is gone; now on net SCL6: U5.18 (SC6)
- net SDL5 is gone; now on net SDA5: U5.15 (SD5)
- net IRQ0: now also U3.28 (IO17); no longer U3.8 (IO32)
- net IRQ1: now also U3.12 (IO27); no longer U3.9 (IO33)
- net IRQ10: now also U3.11 (IO26); no longer U3.28 (IO17)
- net IRQ11: now also U3.10 (IO25); no longer U3.30 (IO18)
- net IRQ12: now also U3.9 (IO33); no longer U3.31 (IO19)
- net IRQ2: now also U3.31 (IO19); no longer U3.10 (IO25)
- net IRQ3: now also U3.30 (IO18); no longer U3.11 (IO26)
- net IRQ4: now also U3.8 (IO32); no longer U3.12 (IO27)
- net IRQ5: now also U3.27 (IO16); no longer U3.13 (IO14)
- net IRQ6: now also U3.7 (IO35); no longer U3.16 (IO13)
- net IRQ8: now also U3.16 (IO13); no longer U3.7 (IO35)
- net IRQ9: now also U3.13 (IO14); no longer U3.27 (IO16)

Commit message: Switch out 22 Ohm resistor 0603 > 0805
Parts:
- R7, R8: footprint Resistor_SMD:R_0402_1005Metric -> 0805W8F220JT5E:0805W8F220JT5E
Changed lines of the file:
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@@
 			)
 		)
-		(property "Footprint" "Resistor_SMD:R_0402_1005Metric"
+		(property "Footprint" "0805W8F220JT5E:0805W8F220JT5E"
 			(at 372.11 39.878 90)
 			(effects
@@
 			)
 		)
-		(property "Footprint" "Resistor_SMD:R_0402_1005Metric"
+		(property "Footprint" "0805W8F220JT5E:0805W8F220JT5E"
 			(at 372.11 38.862 90)
 			(effects
